File: hardware/kicad/battery_protection.kicad_sch (KiCad schematic)
At the start: 4 parts, among them U3 XB8089D0

Commit message: start work on pcb layout
Changed lines of the file:
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@@
 	(paper "A4")
 	(rectangle
-		(start 120.65 69.85)
+		(start 119.38 69.85)
 		(end 161.798 122.174)
 		(stroke
@@
 	(text "Battery Protection (2.9V & 4.25V)"
 		(exclude_from_sim no)
-		(at 137.414 68.834 0)
+		(at 135.636 68.58 0)
 		(effects
 			(font
